Commit message: Ultrasonic Sensors Implementation

File: model/ultrasounds.xacro (robot description, xacro)
@@ -2,8 +2,143 @@
 <robot name="differential_drive_robot" xmlns:xacro="http://www.ros.org/wiki/xacro">
 <!-- Ultrasound 1 Joint-->
-<joint name="ultrasound1_joint" type="fixed">
+<joint name="ultrasonic_joint1" type="fixed">
     <parent link="body_link"/>
-    <child link="laser_frame"/>
-    <origin
+    <child link="ultrasonic_frame1"/>
+    <origin xyz="0.25 0.0 0.045" rpy="0.0 0.0 0.0"/>
 </joint>
+<link name="ultrasonic_frame1">
+    <visual>
+        <geometry>
+            <box size="0.01 0.046 0.031"/>
+        </geometry>
+    </visual>
+    <collision>
+        <geometry>
+            <box size="0.01 0.046 0.031"/>
+        </geometry>
+    </collision>
+</link>
+<gazebo reference="ultrasonic_frame1">
+    <sensor name="ultrasonic1" type="ray">
+        <pose>0 0 0 0 0 0</pose>
+        <visualize>true</visualize>
+        <update_rate>20</update_rate>
+        <ray>
+            <scan>
+                <horizontal>
+                    <samples>20</samples>
+                    <resolution>1</resolution>
+                    <min_angle>-0.2618</min_angle>
+                    <max_angle>0.2618</max_angle>
+                </horizontal>
+            </scan>
+            <range>
+                <min>0.05</min>
+                <max>4.0</max>
+                <resolution>0.01</resolution>
+            </range>
+        </ray>
+        <plugin name="ultrasonic_pub1" filename="libgazebo_ros_ray_sensor.so">
+            <ros>
+                <argument>~/out:=scan</argument>
+            </ros>
+            <output_type>sensor_msgs/LaserScan</output_type>
+            <frame_name>ultrasonic_frame1</frame_name>
+        </plugin>
+    </sensor>
+</gazebo>
+<!-- Ultrasound 2 Joint-->
+<joint name="ultrasonic_joint2" type="fixed">
+    <parent link="body_link"/>
+    <child link="ultrasonic_frame2"/>
+    <origin xyz="0.25 0.075 0.045" rpy="0.0 0.0 0.174533"/>
+</joint>
+<link name="ultrasonic_frame2">
+    <visual>
+        <geometry>
+            <box size="0.01 0.046 0.031"/>
+        </geometry>
+    </visual>
+    <collision>
+        <geometry>
+            <box size="0.01 0.046 0.031"/>
+        </geometry>
+    </collision>
+</link>
+<gazebo reference="ultrasonic_frame2">
+    <sensor name="ultrasonic2" type="ray">
+        <pose>0 0 0 0 0 0</pose>
+        <visualize>true</visualize>
+        <update_rate>20</update_rate>
+        <ray>
+            <scan>
+                <horizontal>
+                    <samples>20</samples>
+                    <resolution>1</resolution>
+                    <min_angle>-0.2618</min_angle>
+                    <max_angle>0.2618</max_angle>
+                </horizontal>
+            </scan>
+            <range>
+                <min>0.05</min>
+                <max>4.0</max>
+                <resolution>0.01</resolution>
+            </range>
+        </ray>
+        <plugin name="ultrasonic_pub2" filename="libgazebo_ros_ray_sensor.so">
+            <ros>
+                <argument>~/out:=scan</argument>
+            </ros>
+            <output_type>sensor_msgs/LaserScan</output_type>
+            <frame_name>ultrasonic_frame2</frame_name>
+        </plugin>
+    </sensor>
+</gazebo>
+<!-- Ultrasound 3 Joint-->
+<joint name="ultrasonic_joint3" type="fixed">
+    <parent link="body_link"/>
+    <child link="ultrasonic_frame3"/>
+    <origin xyz="0.25 -0.075 0.045" rpy="0.0 0.0 -0.174533"/>
+</joint>
+<link name="ultrasonic_frame3">
+    <visual>
+        <geometry>
+            <box size="0.01 0.046 0.031"/>
+        </geometry>
+    </visual>
+    <collision>
+        <geometry>
+            <box size="0.01 0.046 0.031"/>
+        </geometry>
+    </collision>
+</link>
+<gazebo reference="ultrasonic_frame3">
+    <sensor name="ultrasonic3" type="ray">
+        <pose>0 0 0 0 0 0</pose>
+        <visualize>true</visualize>
+        <update_rate>20</update_rate>
+        <ray>
+            <scan>
+                <horizontal>
+                    <samples>20</samples>
+                    <resolution>1</resolution>
+                    <min_angle>-0.2618</min_angle>
+                    <max_angle>0.2618</max_angle>
+                </horizontal>
+            </scan>
+            <range>
+                <min>0.05</min>
+                <max>4.0</max>
+                <resolution>0.01</resolution>
+            </range>
+        </ray>
+        <plugin name="ultrasonic_pub3" filename="libgazebo_ros_ray_sensor.so">
+            <ros>
+                <argument>~/out:=scan</argument>
+            </ros>
+            <output_type>sensor_msgs/LaserScan</output_type>
+            <frame_name>ultrasonic_frame3</frame_name>
+        </plugin>
+    </sensor>
+</gazebo>
 </robot>
