Commit message: Keyboard Teleop and ROS2 Control

File: model/robot.xacro (robot description, xacro)
@@ -1,173 +1,172 @@
 <?xml version="1.0"?>
 <robot name="differential_drive_robot" xmlns:xacro="http://www.ros.org/wiki/xacro">
-<!-- Including other files -->
-<xacro:include filename="ultrasounds.xacro" />
-<!--xacro:include filename="ros2_control.xacro"/-->
-<!-- Body Dimensions -->
-<xacro:property name="body_link_x_dim" value="0.5"/>
-<xacro:property name="body_link_y_dim" value="0.33"/>
-<xacro:property name="body_link_z_dim" value="0.168"/>
-<!-- Wheel Dimensions -->
-<xacro:property name="wheel_link_radius" value="0.1"/>
-<xacro:property name="wheel_link_length" value="0.03"/>
-<xacro:property name="wheel_link_z_location" value="-0.075"/>
-<xacro:property name="wheel_link_y_location" value="0.005"/>
-<!-- Pi Constant -->
-<xacro:property name="pi_const" value="3.14159265"/>
-<!-- Robot Body and Wheel Mass -->
-<xacro:property name="body_mass" value="2.5"/>
-<xacro:property name="wheel_mass" value="0.31"/>
-<!-- Moments of Inertia of the Wheel -->
-<xacro:property name="Iz_wheel" value="${0.5*wheel_mass*wheel_link_radius*wheel_link_radius}"/>
-<xacro:property name="I_wheel"  value="${(1.0/12.0)*wheel_mass*(3*wheel_link_radius*wheel_link_radius+wheel_link_length*wheel_link_length)}"/>
-<xacro:macro name="inertia_wheel">
+  <!-- Including other files -->
+  <xacro:include filename="ultrasounds.xacro" />
+  <xacro:include filename="ros2_control.xacro" />
+  <!-- Body Dimensions -->
+  <xacro:property name="body_link_x_dim" value="0.5"/>
+  <xacro:property name="body_link_y_dim" value="0.33"/>
+  <xacro:property name="body_link_z_dim" value="0.168"/>
+  <!-- Wheel Dimensions -->
+  <xacro:property name="wheel_link_radius" value="0.1"/>  <!-- 10 cm radio -->
+  <xacro:property name="wheel_link_length" value="0.03"/>
+  <xacro:property name="wheel_link_z_location" value="-0.075"/>
+  <xacro:property name="wheel_link_y_location" value="0.005"/>
+  <!-- Pi Constant -->
+  <xacro:property name="pi_const" value="3.14159265"/>
+  <!-- Robot Body and Wheel Mass -->
+  <xacro:property name="body_mass" value="3.5"/>
+  <xacro:property name="wheel_mass" value="0.35"/>
+  <!-- Moments of Inertia of the Wheel -->
+  <xacro:property name="Iz_wheel" value="${0.5*wheel_mass*wheel_link_radius*wheel_link_radius}"/>
+  <xacro:property name="I_wheel"  value="${(1.0/12.0)*wheel_mass*(3*wheel_link_radius*wheel_link_radius+wheel_link_length*wheel_link_length)}"/>
+  <xacro:macro name="inertia_wheel">
     <inertial>
-        <origin xyz="0.0 0.0 0.0" rpy="0.0 0.0 0.0"/>
-        <mass value="${wheel_mass}"/>
-        <inertia ixx="${I_wheel}" ixy="0.0" ixz="0.0" iyy="${I_wheel}" iyz="0.0" izz="${Iz_wheel}" />
+      <origin xyz="0.0 0.0 0.0" rpy="0.0 0.0 0.0"/>
+      <mass value="${wheel_mass}"/>
+      <inertia ixx="${I_wheel}" ixy="0.0" ixz="0.0"
+               iyy="${I_wheel}" iyz="0.0" izz="${Iz_wheel}" />
     </inertial>
-</xacro:macro>
-<!-- Extra Gazebo Options -->
-<xacro:include filename="$(find lawn_robot)/model/robot.gazebo" />
-<!-- ########################################## -->
-<!--         Links and Joints Definition        -->
-<!-- ########################################## -->
-<!-- Dummy link, otherwise Gazebo will complain -->
-<link name="dummy">
-</link>
-<joint name="dummy_joint" type="fixed">
+  </xacro:macro>
+  <!-- Extra Gazebo Options -->
+  <xacro:include filename="$(find lawn_robot)/model/robot.gazebo" />
+  <!-- Dummy link, otherwise Gazebo will complain -->
+  <link name="dummy"/>
+  <joint name="dummy_joint" type="fixed">
     <parent link="dummy"/>
     <child link="body_link"/>
-</joint>
-<!-- ########################################## -->
-<!--           Body Link of the robot           -->
-<!-- ########################################## -->
-<link name="body_link">
+  </joint>
+  <!-- BODY LINK -->
+  <link name="body_link">
     <visual>
-        <geometry>
-            <box size="${body_link_x_dim} ${body_link_y_dim} ${body_link_z_dim}" />
-        </geometry>
-        <origin xyz="0.0 0.0 0.0" rpy="0.0 0.0 0.0"/>
+      <geometry>
+        <box size="${body_link_x_dim} ${body_link_y_dim} ${body_link_z_dim}" />
+      </geometry>
+      <origin xyz="0 0 0" rpy="0 0 0"/>
     </visual>
     <collision>
-        <geometry>
-            <box size="${body_link_x_dim} ${body_link_y_dim} ${body_link_z_dim}" />
-        </geometry>
-        <origin xyz="0.0 0.0 0.0" rpy="0.0 0.0 0.0"/>
+      <geometry>
+        <box size="${body_link_x_dim} ${body_link_y_dim} ${body_link_z_dim}" />
+      </geometry>
+      <origin xyz="0 0 0" rpy="0 0 0"/>
     </collision>
     <inertial>
-        <origin xyz="0.0 0.0 0.0" rpy="0.0 0.0 0.0"/>
-        <mass value="${body_mass}" />
-    <inertia
-    ixx="${(1.0/12.0)*body_mass*(body_link_y_dim*body_link_y_dim+body_link_z_dim*body_link_z_dim)}"
-    ixy="0" ixz="0"
-    iyy="${(1.0/12.0)*body_mass*(body_link_x_dim*body_link_x_dim+body_link_z_dim*body_link_z_dim)}"
-    iyz="0"
-    izz="${(1.0/12.0)*body_mass*(body_link_y_dim*body_link_y_dim+body_link_x_dim*body_link_x_dim)}" />
+      <origin xyz="0 0 0" rpy="0 0 0"/>
+      <mass value="${body_mass}" />
+      <inertia
+        ixx="${(1.0/12.0)*body_mass*(body_link_y_dim*body_link_y_dim+body_link_z_dim*body_link_z_dim)}"
+        ixy="0" ixz="0"
+        iyy="${(1.0/12.0)*body_mass*(body_link_x_dim*body_link_x_dim+body_link_z_dim*body_link_z_dim)}"
+        iyz="0"
+        izz="${(1.0/12.0)*body_mass*(body_link_y_dim*body_link_y_dim+body_link_x_dim*body_link_x_dim)}" />
     </inertial>
-</link>
-<!-- ########################################## -->
-<!--        Back Right Wheel of the robot       -->
-<!-- ########################################## -->
-<joint name="wheel1_joint" type="continuous">
+  </link>
+  <!-- BACK RIGHT WHEEL -->
+  <joint name="wheel1_joint" type="continuous">
     <parent link="body_link"/>
     <child link="wheel1_link"/>
-    <origin xyz="${-body_link_x_dim/2+0.4*wheel_link_radius} ${-body_link_y_dim/2-((wheel_link_length/2)+wheel_link_y_location)} ${wheel_link_z_location}" rpy="0.0 0.0 0.0"/>
+    <origin xyz="${-body_link_x_dim/2+0.4*wheel_link_radius}
+                 ${-body_link_y_dim/2-((wheel_link_length/2)+wheel_link_y_location)}
+                 ${wheel_link_z_location}"
+            rpy="0 0 0"/>
     <axis xyz="0 1 0"/>
     <limit effort="1000" velocity="1000"/>
-    <dynamics damping="1.0" friction="1.0" />
-</joint>
-<link name="wheel1_link">
+    <dynamics damping="0.05" friction="0.05" />
+  </joint>
+  <link name="wheel1_link">
     <visual>
-        <origin xyz="0.0 0.0 0.0" rpy="${pi_const/2} 0 0"/>
-        <geometry>
-            <cylinder radius="${wheel_link_radius}" length="${wheel_link_length}"/>
-        </geometry>
+      <origin xyz="0 0 0" rpy="${pi_const/2} 0 0"/>
+      <geometry>
+        <cylinder radius="${wheel_link_radius}" length="${wheel_link_length}"/>
+      </geometry>
     </visual>
     <collision>
-        <origin xyz="0.0 0.0 0.0" rpy="${pi_const/2} 0 0"/>
-        <geometry>
-            <cylinder radius="${wheel_link_radius}" length="${wheel_link_length}"/>
-        </geometry>
+      <origin xyz="0 0 0" rpy="0 0 0"/>
+      <geometry>
+        <sphere radius="${wheel_link_radius}"/>
+      </geometry>
     </collision>
     <xacro:inertia_wheel />
-</link>
-<!-- ########################################## -->
-<!--        Back Left Wheel of the robot       -->
-<!-- ########################################## -->
-<joint name="wheel2_joint" type="continuous">
+  </link>
+  <!-- BACK LEFT WHEEL -->
+  <joint name="wheel2_joint" type="continuous">
     <parent link="body_link"/>
     <child link="wheel2_link"/>
-    <origin xyz="${-body_link_x_dim/2+0.4*wheel_link_radius} ${body_link_y_dim/2+((wheel_link_length/2)+wheel_link_y_location)} ${wheel_link_z_location}" rpy="0.0 0.0 0.0"/>
+    <origin xyz="${-body_link_x_dim/2+0.4*wheel_link_radius}
+                 ${body_link_y_dim/2+((wheel_link_length/2)+wheel_link_y_location)}
+                 ${wheel_link_z_location}"
+            rpy="0 0 0"/>
     <axis xyz="0 1 0"/>
     <limit effort="1000" velocity="1000"/>
-    <dynamics damping="1.0" friction="1.0" />
-</joint>
-<link name="wheel2_link">
+    <dynamics damping="0.05" friction="0.05" />
+  </joint>
+  <link name="wheel2_link">
     <visual>
-        <origin xyz="0.0 0.0 0.0" rpy="${pi_const/2} 0 0"/>
-        <geometry>
-            <cylinder radius="${wheel_link_radius}" length="${wheel_link_length}"/>
-        </geometry>
+      <origin xyz="0 0 0" rpy="${pi_const/2} 0 0"/>
+      <geometry>
+        <cylinder radius="${wheel_link_radius}" length="${wheel_link_length}"/>
+      </geometry>
     </visual>
     <collision>
-        <origin xyz="0.0 0.0 0.0" rpy="${pi_const/2} 0 0"/>
-        <geometry>
-            <cylinder radius="${wheel_link_radius}" length="${wheel_link_length}"/>
-        </geometry>
+      <origin xyz="0 0 0" rpy="0 0 0"/>
+      <geometry>
+        <sphere radius="${wheel_link_radius}"/>
+      </geometry>
     </collision>
     <xacro:inertia_wheel />
-</link>
-<!-- ########################################## -->
-<!--        Front Right Wheel of the robot       -->
-<!-- ########################################## -->
-<joint name="wheel3_joint" type="continuous">
+  </link>
+  <!-- FRONT RIGHT WHEEL -->
+  <joint name="wheel3_joint" type="continuous">
     <parent link="body_link"/>
     <child link="wheel3_link"/>
-    <origin xyz="${body_link_x_dim/2-0.4*wheel_link_radius} ${-body_link_y_dim/2-((wheel_link_length/2)+wheel_link_y_location)} ${wheel_link_z_location}" rpy="0.0 0.0 0.0"/>
+    <origin xyz="${body_link_x_dim/2-0.4*wheel_link_radius}
+                 ${-body_link_y_dim/2-((wheel_link_length/2)+wheel_link_y_location)}
+                 ${wheel_link_z_location}"
+            rpy="0 0 0"/>
     <axis xyz="0 1 0"/>
     <limit effort="1000" velocity="1000"/>
-    <dynamics damping="1.0" friction="1.0" />
-</joint>
-<link name="wheel3_link">
+    <dynamics damping="0.05" friction="0.05" />
+  </joint>
+  <link name="wheel3_link">
     <visual>
-        <origin xyz="0.0 0.0 0.0" rpy="${pi_const/2} 0 0"/>
-        <geometry>
-            <cylinder radius="${wheel_link_radius}" length="${wheel_link_length}"/>
-        </geometry>
+      <origin xyz="0 0 0" rpy="${pi_const/2} 0 0"/>
+      <geometry>
+        <cylinder radius="${wheel_link_radius}" length="${wheel_link_length}"/>
+      </geometry>
     </visual>
     <collision>
-        <origin xyz="0.0 0.0 0.0" rpy="${pi_const/2} 0 0"/>
-        <geometry>
-            <cylinder radius="${wheel_link_radius}" length="${wheel_link_length}"/>
-        </geometry>
+      <origin xyz="0 0 0" rpy="0 0 0"/>
+      <geometry>
+        <sphere radius="${wheel_link_radius}"/>
+      </geometry>
     </collision>
     <xacro:inertia_wheel />
-</link>
-<!-- ########################################## -->
-<!--        Front Right Wheel of the robot       -->
-<!-- ########################################## -->
-<joint name="wheel4_joint" type="continuous">
+  </link>
+  <!-- FRONT LEFT WHEEL -->
+  <joint name="wheel4_joint" type="continuous">
     <parent link="body_link"/>
     <child link="wheel4_link"/>
-    <origin xyz="${body_link_x_dim/2-0.4*wheel_link_radius} ${body_link_y_dim/2+((wheel_link_length/2)+wheel_link_y_location)} ${wheel_link_z_location}" rpy="0.0 0.0 0.0"/>
+    <origin xyz="${body_link_x_dim/2-0.4*wheel_link_radius}
+                 ${body_link_y_dim/2+((wheel_link_length/2)+wheel_link_y_location)}
+                 ${wheel_link_z_location}"
+            rpy="0 0 0"/>
     <axis xyz="0 1 0"/>
     <limit effort="1000" velocity="1000"/>
-    <dynamics damping="1.0" friction="1.0" />
-</joint>
-<link name="wheel4_link">
+    <dynamics damping="0.05" friction="0.05" />
+  </joint>
+  <link name="wheel4_link">
     <visual>
-        <origin xyz="0.0 0.0 0.0" rpy="${pi_const/2} 0 0"/>
-        <geometry>
-            <cylinder radius="${wheel_link_radius}" length="${wheel_link_length}"/>
-        </geometry>
+      <origin xyz="0 0 0" rpy="${pi_const/2} 0 0"/>
+      <geometry>
+        <cylinder radius="${wheel_link_radius}" length="${wheel_link_length}"/>
+      </geometry>
     </visual>
     <collision>
-        <origin xyz="0.0 0.0 0.0" rpy="${pi_const/2} 0 0"/>
-        <geometry>
-            <cylinder radius="${wheel_link_radius}" length="${wheel_link_length}"/>
-        </geometry>
+      <origin xyz="0 0 0" rpy="0 0 0"/>
+      <geometry>
+        <sphere radius="${wheel_link_radius}"/>
+      </geometry>
     </collision>
     <xacro:inertia_wheel />
-</link>
+  </link>
 </robot>

File: model/ros2_control.xacro (robot description, xacro)
@@ -1,38 +1,104 @@
 <?xml version="1.0"?>
-<robot>
-<gazebo reference="body_link">
-    <mu1>0.2</mu1>
-    <mu2>0.2</mu2>
-    <material>
-        Gazebo/Grey
-    </material>
-</gazebo>
-<gazebo reference="wheel1_link">
-    <mu1>0.2</mu1>
-    <mu2>0.2</mu2>
-    <material>
-        Gazebo/DarkGrey
-    </material>
-</gazebo>
-<gazebo reference="wheel2_link">
-    <mu1>0.2</mu1>
-    <mu2>0.2</mu2>
-    <material>
-        Gazebo/DarkGrey
-    </material>
-</gazebo>
-<gazebo reference="wheel3_link">
-    <mu1>0.2</mu1>
-    <mu2>0.2</mu2>
-    <material>
-        Gazebo/DarkGrey
-    </material>
-</gazebo>
-<gazebo reference="wheel4_link">
-    <mu1>0.2</mu1>
-    <mu2>0.2</mu2>
-    <material>
-        Gazebo/DarkGrey
-    </material>
-</gazebo>
+<robot xmlns:xacro="http://www.ros.org/wiki/xacro">
+  <!-- ===================== -->
+  <!--  Datos del motor      -->
+  <!--  25GA370-12V-100RPM   -->
+  <!-- ===================== -->
+  <!-- Velocidad máxima en RPM -->
+  <xacro:property name="motor_rpm_max" value="100"/>
+  <!-- rad/s = RPM * 2*pi / 60 -->
+  <xacro:property name="motor_rad_s_max" value="${motor_rpm_max * 2.0 * 3.14159265 / 60.0}"/>
+  <!-- ===================== -->
+  <!--  ros2_control system  -->
+  <!-- ===================== -->
+  <ros2_control name="lawn_robot_control" type="system">
+    <hardware>
+      <plugin>gazebo_ros2_control/GazeboSystem</plugin>
+    </hardware>
+    <!-- Rueda 1 -->
+    <joint name="wheel1_joint">
+      <command_interface name="velocity">
+        <param name="min">${-motor_rad_s_max}</param>
+        <param name="max">${motor_rad_s_max}</param>
+      </command_interface>
+      <state_interface name="velocity"/>
+      <state_interface name="position"/>
+    </joint>
+    <!-- Rueda 2 -->
+    <joint name="wheel2_joint">
+      <command_interface name="velocity">
+        <param name="min">${-motor_rad_s_max}</param>
+        <param name="max">${motor_rad_s_max}</param>
+      </command_interface>
+      <state_interface name="velocity"/>
+      <state_interface name="position"/>
+    </joint>
+    <!-- Rueda 3 -->
+    <joint name="wheel3_joint">
+      <command_interface name="velocity">
+        <param name="min">${-motor_rad_s_max}</param>
+        <param name="max">${motor_rad_s_max}</param>
+      </command_interface>
+      <state_interface name="velocity"/>
+      <state_interface name="position"/>
+    </joint>
+    <!-- Rueda 4 -->
+    <joint name="wheel4_joint">
+      <command_interface name="velocity">
+        <param name="min">${-motor_rad_s_max}</param>
+        <param name="max">${motor_rad_s_max}</param>
+      </command_interface>
+      <state_interface name="velocity"/>
+      <state_interface name="position"/>
+    </joint>
+  </ros2_control>
+  <!-- ===================== -->
+  <!--   Transmisiones       -->
+  <!-- ===================== -->
+  <transmission name="wheel1_trans">
+    <type>transmission_interface/SimpleTransmission</type>
+    <actuator name="wheel1_motor">
+      <mechanicalReduction>1</mechanicalReduction>
+    </actuator>
+    <joint name="wheel1_joint">
+      <hardwareInterface>hardware_interface/velocity</hardwareInterface>
+    </joint>
+  </transmission>
+  <transmission name="wheel2_trans">
+    <type>transmission_interface/SimpleTransmission</type>
+    <actuator name="wheel2_motor">
+      <mechanicalReduction>1</mechanicalReduction>
+    </actuator>
+    <joint name="wheel2_joint">
+      <hardwareInterface>hardware_interface/velocity</hardwareInterface>
+    </joint>
+  </transmission>
+  <transmission name="wheel3_trans">
+    <type>transmission_interface/SimpleTransmission</type>
+    <actuator name="wheel3_motor">
+      <mechanicalReduction>1</mechanicalReduction>
+    </actuator>
+    <joint name="wheel3_joint">
+      <hardwareInterface>hardware_interface/velocity</hardwareInterface>
+    </joint>
+  </transmission>
+  <transmission name="wheel4_trans">
+    <type>transmission_interface/SimpleTransmission</type>
+    <actuator name="wheel4_motor">
+      <mechanicalReduction>1</mechanicalReduction>
+    </actuator>
+    <joint name="wheel4_joint">
+      <hardwareInterface>hardware_interface/velocity</hardwareInterface>
+    </joint>
+  </transmission>
+  <!-- ===================== -->
+  <!--  Plugin Gazebo        -->
+  <!-- ===================== -->
+  <gazebo>
+    <plugin name="gazebo_ros2_control" filename="libgazebo_ros2_control.so">
+      <robot_param>robot_description</robot_param>
+      <robot_param_node>robot_state_publisher</robot_param_node>
+      <parameters>$(find lawn_robot)/config/ros2_controller.yaml</parameters>
+    </plugin>
+  </gazebo>
 </robot>
